File: host_pcb/host_pcb.kicad_pcb (KiCad board)
At the start: 2 copper layers, 15 parts, among them P1 CONN_4, P2 CONN_4, U1 STM32F407VG, U2 ULN2803A, U3 ULN2803A, U4 ULN2803A, U5 LM2596, U6 SN65HVD230, U7 ULN2803A

Commit message: WIP: host PCB
Parts:
- removed U7: ULN2803A, SO20L
- U5: footprint SOT353 -> TO263-5
- moved JP1 15.3 mm to (153.4, 83.9), turned to 90 degrees
- moved U5 12.0 mm to (113.6, 97.7), turned to 90 degrees
- moved R1 4.36 mm to (147.1, 85.1), turned to 0 degrees
Other:
- board outline added: 122.2 x 86.9 mm

Commit message: WIP: host pcb
Parts:
- added C10: CSMALL, SM0805, F.Cu at (120.6, 163.2)
- added C11: CSMALL, SM0805, F.Cu at (123.8, 155.2)
- added C12: CSMALL, SM0805, F.Cu at (129.1, 154.6)
- added C13: CSMALL, SM0805, F.Cu at (135.6, 154.9)
- added C14: CSMALL, SM0805, F.Cu at (143.5, 158.5)
- added C15: CSMALL, SM0805, F.Cu at (140.0, 162.9)
- added C16: CSMALL, SM0805, F.Cu at (127.5, 164.9)
- added C3: C, SM1812, F.Cu at (151.7, 161.1)
- added C4: C, SM1812, F.Cu at (135.6, 169.4)
- added C5: C, SM1812, F.Cu at (121.3, 169.7)
- added C6: C, SM1812, F.Cu at (117.2, 154.2)
- added C7: C, SM1812, F.Cu at (132.4, 161.0)
- added C8: CSMALL, SM0805, F.Cu at (118.7, 158.9)
- added C9: CSMALL, SM0805, F.Cu at (146.6, 154.2)
- added D2: LED, SM0805, F.Cu at (120.2, 146.9)
- added D3: LED, SM0805, F.Cu at (135.1, 147.8)
- added D4: LED, SM0805, F.Cu at (137.3, 147.8)
- added D5: LED, SM0805, F.Cu at (131.9, 147.8)
- added D6: LED, SM0805, F.Cu at (128.8, 147.8)
- added P10: BTNS, pin_array_4x2, F.Cu at (99.7, 126.0)
- added P11: PWR_IN, PIN_ARRAY_2X1, F.Cu at (117.4, 80.2)
- added P12: PWR_OUT, PIN_ARRAY_2X1, F.Cu at (184.0, 143.8)
- added P13: OUT_1, pin_array_4x2, F.Cu at (181.3, 137.3)
- added P14: OUT_2, pin_array_4x2, F.Cu at (181.0, 130.9)
- added P15: OUT_3, pin_array_4x2, F.Cu at (180.7, 124.2)
- added P3: RST, PIN_ARRAY_2X1, F.Cu at (99.7, 118.7)
- added P4: LCD, pin_array_8x2, F.Cu at (134.3, 106.1)
- added P5: SWD, PIN_ARRAY-6X1, F.Cu at (171.2, 97.7)
- added P6: UART2, PIN_ARRAY_4x1, F.Cu at (177.9, 95.2)
- added P7: IN_1, pin_array_4x2, F.Cu at (160.7, 146.7)
- added P8: IN_2, pin_array_4x2, F.Cu at (149.5, 146.6)
- added P9: IN_3, pin_array_4x2, F.Cu at (171.5, 146.7)
- added R2: R, SM0805, F.Cu at (120.8, 131.2)
- added R3: R, SM0805, F.Cu at (123.8, 146.2)
- added R4: R, SM0805, F.Cu at (134.9, 143.1)
- added R5: R, SM0805, F.Cu at (137.4, 142.9)
- added R6: R, SM0805, F.Cu at (131.7, 142.9)
- added R7: R, SM0805, F.Cu at (128.8, 143.1)
- added SW1: SW_PUSH, SW_PUSH_SMALL, F.Cu at (112.0, 112.0)
- added SW2: SW_PUSH, SW_PUSH_SMALL, F.Cu at (112.2, 121.1)
- added SW3: SW_PUSH, SW_PUSH_SMALL, F.Cu at (112.2, 129.8)
- added SW4: SW_PUSH, SW_PUSH_SMALL, F.Cu at (112.3, 139.7)
- added SW5: SW_PUSH, SW_PUSH_SMALL, F.Cu at (100.5, 112.1)
- added X1: CRYSTAL, HC-49V, F.Cu at (123.5, 124.3)
- P1, P2: value CONN_4 -> RJ45
- moved U6 1.91 mm to (132.3, 89.8), turned to 0 degrees
Connections:
- JP1 pad 2: canl -> canh
- P1 pad 2: canh -> 12v
- P1 pad 3: canl -> Net-<P1-Pad3>
- P1 pad 5: (no net) -> vss
- P1 pad 6: (no net) -> Net-<P1-Pad6>
- P1 pad 7: (no net) -> canh
- P1 pad 8: (no net) -> canl
- P2 pad 2: canh -> 12v
- P2 pad 3: canl -> Net-<P2-Pad3>
- P2 pad 5: (no net) -> vss
- P2 pad 6: (no net) -> Net-<P2-Pad6>
- P2 pad 7: (no net) -> canh
- P2 pad 8: (no net) -> canl
- R1 pad 1: canh -> canl
- U1 pad 1: Net-<U1-Pad1> -> /ld2
- U1 pad 12: Net-<U1-Pad12> -> oscin
- U1 pad 13: Net-<U1-Pad13> -> oscout
- U1 pad 15: Net-<U1-Pad15> -> /ld7
- U1 pad 16: Net-<U1-Pad16> -> /lrs
- U1 pad 17: Net-<U1-Pad17> -> /lrw
- U1 pad 18: Net-<U1-Pad18> -> /le
- U1 pad 19: Net-<U1-Pad19> -> 3v3
- U1 pad 2: Net-<U1-Pad2> -> /ld3
- U1 pad 3: Net-<U1-Pad3> -> /ld4
- U1 pad 4: Net-<U1-Pad4> -> /ld5
- U1 pad 49: Net-<U1-Pad49> -> Net-<C6-Pad1>
- U1 pad 5: Net-<U1-Pad5> -> /ld6
- U1 pad 56: Net-<U1-Pad56> -> /a1
- U1 pad 57: Net-<U1-Pad57> -> /a2
- U1 pad 58: Net-<U1-Pad58> -> /a3
- U1 pad 59: Net-<U1-Pad59> -> /a4
- U1 pad 60: Net-<U1-Pad60> -> /a5
- U1 pad 61: Net-<U1-Pad61> -> /a6
- U1 pad 62: Net-<U1-Pad62> -> /a7
- U1 pad 63: Net-<U1-Pad63> -> /a8
- U1 pad 64: Net-<U1-Pad64> -> /a9
- U1 pad 65: Net-<U1-Pad65> -> /a10
- U1 pad 66: Net-<U1-Pad66> -> /a11
- U1 pad 67: Net-<U1-Pad67> -> /a12
- U1 pad 68: Net-<U1-Pad68> -> /a13
- U1 pad 69: Net-<U1-Pad69> -> /a14
- U1 pad 7: Net-<U1-Pad7> -> /ld0
- U1 pad 70: Net-<U1-Pad70> -> /a15
- U1 pad 71: Net-<U1-Pad71> -> /a16
- U1 pad 73: Net-<U1-Pad73> -> Net-<C7-Pad1>
- U1 pad 77: Net-<U1-Pad77> -> /a17
- U1 pad 78: Net-<U1-Pad78> -> /a18
- U1 pad 79: Net-<U1-Pad79> -> /a19
- U1 pad 8: Net-<U1-Pad8> -> /ld1
- U1 pad 80: Net-<U1-Pad80> -> /a20
- U1 pad 81: Net-<U1-Pad81> -> /a21
- U1 pad 82: Net-<U1-Pad82> -> /a22
- U1 pad 83: Net-<U1-Pad83> -> /a23
- U1 pad 84: Net-<U1-Pad84> -> /a24
- U1 pad 85: Net-<U1-Pad85> -> led0
- U1 pad 86: Net-<U1-Pad86> -> led1
- U1 pad 87: Net-<U1-Pad87> -> led2
- U1 pad 88: Net-<U1-Pad88> -> led3
- U1 pad 89: Net-<U1-Pad89> -> traceswo
- U1 pad 90: Net-<U1-Pad90> -> btn0
- U1 pad 91: Net-<U1-Pad91> -> btn1
- U1 pad 92: Net-<U1-Pad92> -> btn2
- U1 pad 93: Net-<U1-Pad93> -> btn3
- U2 pad 10: Net-<U2-Pad10> -> 12v
- U2 pad 11: Net-<U2-Pad11> -> /d1
- U2 pad 12: Net-<U2-Pad12> -> /d2
- U2 pad 13: Net-<U2-Pad13> -> /d3
- U2 pad 14: Net-<U2-Pad14> -> /d4
- U2 pad 15: Net-<U2-Pad15> -> /d5
- U2 pad 16: Net-<U2-Pad16> -> /d6
- U2 pad 17: Net-<U2-Pad17> -> /d7
- U2 pad 18: Net-<U2-Pad18> -> /d8
- U3 pad 10: Net-<U3-Pad10> -> 12v
- U3 pad 11: Net-<U3-Pad11> -> /d9
- U3 pad 12: Net-<U3-Pad12> -> /d10
- U3 pad 13: Net-<U3-Pad13> -> /d11
- U3 pad 14: Net-<U3-Pad14> -> /d12
- U3 pad 15: Net-<U3-Pad15> -> /d13
- U3 pad 16: Net-<U3-Pad16> -> /d14
- U3 pad 17: Net-<U3-Pad17> -> /d15
- U3 pad 18: Net-<U3-Pad18> -> /d16
- U4 pad 10: Net-<U4-Pad10> -> 12v
- U4 pad 11: Net-<U4-Pad11> -> /d17
- U4 pad 12: Net-<U4-Pad12> -> /d18
- U4 pad 13: Net-<U4-Pad13> -> /d19
- U4 pad 14: Net-<U4-Pad14> -> /d20
- U4 pad 15: Net-<U4-Pad15> -> /d21
- U4 pad 16: Net-<U4-Pad16> -> /d22
- U4 pad 17: Net-<U4-Pad17> -> /d23
- U4 pad 18: Net-<U4-Pad18> -> /d24
