File: host_pcb/host_pcb.sch (KiCad schematic (older format))
At the start: 15 parts, among them P1 CONN_4, P2 CONN_4, U1 STM32F407VG, U2 ULN2803A, U3 ULN2803A, U4 ULN2803A, U5 LM2596, U6 SN65HVD230, U7 ULN2803A

Commit message: WIP: host PCB
Parts:
- removed U7: ULN2803A, MODULE, symbol ULN2803A
Changed lines of the file:
@@
 Wire Wire Line
 	2500 1850 2500 1750
-$Comp
-L ULN2803A U7
-U 1 1 52656480
-P 5750 6250
-F 0 "U7" H 5750 6150 50  0000 C CNN
-F 1 "ULN2803A" H 5750 6350 50  0000 C CNN
-F 2 "MODULE" H 5750 6250 50  0001 C CNN
-F 3 "DOCUMENTATION" H 5750 6250 50  0001 C CNN
-	1    5750 6250
-	1    0    0    -1
-$EndComp
 $EndSCHEMATC

Commit message: WIP: host pcb
Parts:
- added C10, C11, C12, C13, C14, C15, C16, C8, C9: CSMALL, symbol CSMALL
- added C3, C4: 20pF, symbol C
- added C5: 1uF, symbol C
- added C6, C7: C, symbol C
- added D2, D3, D4, D5, D6: LED, symbol LED
- added P10: BTNS, symbol CONN_4X2
- added P11: PWR_IN, symbol CONN_2
- added P12: PWR_OUT, symbol CONN_2
- added P13: OUT_1, symbol CONN_8
- added P14: OUT_2, symbol CONN_8
- added P15: OUT_3, symbol CONN_8
- added P3: RST, symbol CONN_2
- added P4: LCD, symbol CONN_8X2
- added P5: SWD, symbol CONN_6
- added P6: UART2, symbol CONN_4
- added P7: IN_1, symbol CONN_8
- added P8: IN_2, symbol CONN_8
- added P9: IN_3, symbol CONN_8
- added R2, R3, R4, R5, R6, R7: R, symbol R
- added SW1: SW_RST, symbol SW_PUSH
- added SW2: SW_U0, symbol SW_PUSH
- added SW3: SW_U1, symbol SW_PUSH
- added SW4: SW_U2, symbol SW_PUSH
- added SW5: SW_U3, symbol SW_PUSH
- added X1: 8MHz, symbol CRYSTAL
- C1: value CP1 -> 680uF
- C2: value CP1 -> 330uF
- JP1: value JUMPER -> CAN_TERM
- L1: value INDUCTOR -> 33uH
- P1, P2: value CONN_4 -> RJ45; symbol CONN_4 -> CONN_8
Connections:
- net labels added: a1, a10, a11, a12, a13, a14, a15, a16, a17, a18, a19, a2, a20, a21, a22, a23, a24, a3, a4, a5, a6, a7, a8, a9, btn0, btn1, btn2, btn3, d1, d10, d11, d12, d13, d14, d15, d16, d17, d18, d19, d2, d20, d21, d22, d23, d24, d3, d4, d5, d6, d7, d8, d9, ld0, ld1, ld2, ld3, ld4, ld5, ld6, ld7, le, led0, led1, led2, led3, lrs, lrw, oscin, oscout, traceswo, uart2_rx, uart2_tx
- wire segments 43 -> 77
- no-connect marks 1 -> 8
Other:
- moved on the sheet: U6

Commit message: WIP: host PCB
Parts:
- R2: value R -> 220
Changed lines of the file:
@@
 P 1400 3250
 F 0 "R2" V 1480 3250 50  0000 C CNN
-F 1 "R" V 1400 3250 50  0000 C CNN
+F 1 "220" V 1400 3250 50  0000 C CNN
 F 2 "" H 1400 3250 60  0000 C CNN
 F 3 "" H 1400 3250 60  0000 C CNN

Commit message: WIP: host pcb
Parts:
- removed P3: RST, symbol CONN_2
- C10, C11, C12, C14, C16, C8, C9: value CSMALL -> 100nF
- C13: value CSMALL -> 4.7uF
- C15: value CSMALL -> 1uF
- C6, C7: value C -> 2.2uF
- D1: value DIODESCH -> MURS320T3G
- P10: symbol CONN_4X2 -> CONN_5X2
- P13, P14, P15, P7, P8, P9: symbol CONN_8 -> CONN_8X2
- R1: value R -> 120
- R4, R5, R6, R7: value R -> 770
Connections:
- wire segments 77 -> 78
- no-connect marks 8 -> 13
Changed lines of the file:
@@
 P 2500 1550
 F 0 "D1" H 2500 1650 40  0000 C CNN
-F 1 "DIODESCH" H 2500 1450 40  0000 C CNN
+F 1 "MURS320T3G" H 2500 1450 40  0000 C CNN
 F 2 "" H 2500 1550 60  0001 C CNN
 F 3 "" H 2500 1550 60  0001 C CNN
@@
 P 2850 7400
 F 0 "R1" V 2930 7400 50  0000 C CNN
-F 1 "R" V 2850 7400 50  0000 C CNN
+F 1 "120" V 2850 7400 50  0000 C CNN
 F 2 "" H 2850 7400 60  0001 C CNN
 F 3 "" H 2850 7400 60  0001 C CNN
@@
 P 6550 5600
 F 0 "C6" H 6600 5700 50  0000 L CNN
-F 1 "C" H 6600 5500 50  0000 L CNN
+F 1 "2.2uF" H 6600 5500 50  0000 L CNN
 F 2 "" H 6550 5600 60  0000 C CNN
 F 3 "" H 6550 5600 60  0000 C CNN
@@
 P 7900 2250
 F 0 "C7" H 7950 2350 50  0000 L CNN
-F 1 "C" H 7950 2150 50  0000 L CNN
+F 1 "2.2uF" H 7950 2150 50  0000 L CNN
 F 2 "" H 7900 2250 60  0000 C CNN
 F 3 "" H 7900 2250 60  0000 C CNN
@@
 	1    1400 4300
 	1    0    0    -1
-$EndComp
-$Comp
-L CONN_2 P3
-U 1 1 52669C6D
-P 800 4200
-F 0 "P3" V 750 4200 40  0000 C CNN
-F 1 "RST" V 850 4200 40  0000 C CNN
-F 2 "" H 800 4200 60  0000 C CNN
-F 3 "" H 800 4200 60  0000 C CNN
-	1    800  4200
-	-1   0    0    1
 $EndComp
 $Comp
@@
 	10150 4650 10250 4750
 $Comp
-L CONN_8 P13
+L CONN_8X2 P13
 U 1 1 5266A7BC
-P 11050 2600
-F 0 "P13" V 11000 2600 60  0000 C CNN
-F 1 "OUT_1" V 11100 2600 60  0000 C CNN
-F 2 "" H 11050 2600 60  0000 C CNN
-F 3 "" H 11050 2600 60  0000 C CNN
-	1    11050 2600
+P 11100 2600
+F 0 "P13" V 11050 2600 60  0000 C CNN
+F 1 "OUT_1" V 11150 2600 60  0000 C CNN
+F 2 "" H 11100 2600 60  0000 C CNN
+F 3 "" H 11100 2600 60  0000 C CNN
+	1    11100 2600
 	1    0    0    1
 $EndComp
@@
 	10600 2850 10700 2950
 $Comp
-L CONN_8 P14
+L CONN_8X2 P14
 U 1 1 5266A7F4
-P 11050 3850
-F 0 "P14" V 11000 3850 60  0000 C CNN
-F 1 "OUT_2" V 11100 3850 60  0000 C CNN
-F 2 "" H 11050 3850 60  0000 C CNN
-F 3 "" H 11050 3850 60  0000 C CNN
-	1    11050 3850
+P 11100 3850
+F 0 "P14" V 11050 3850 60  0000 C CNN
+F 1 "OUT_2" V 11150 3850 60  0000 C CNN
+F 2 "" H 11100 3850 60  0000 C CNN
+F 3 "" H 11100 3850 60  0000 C CNN
+	1    11100 3850
 	1    0    0    1
 $EndComp
@@
 	10600 4100 10700 4200
 $Comp
-L CONN_8 P15
+L CONN_8X2 P15
 U 1 1 5266A972
-P 11050 5100
-F 0 "P15" V 11000 5100 60  0000 C CNN
-F 1 "OUT_3" V 11100 5100 60  0000 C CNN
-F 2 "" H 11050 5100 60  0000 C CNN
-F 3 "" H 11050 5100 60  0000 C CNN
-	1    11050 5100
+P 11100 5100
+F 0 "P15" V 11050 5100 60  0000 C CNN
+F 1 "OUT_3" V 11150 5100 60  0000 C CNN
+F 2 "" H 11100 5100 60  0000 C CNN
+F 3 "" H 11100 5100 60  0000 C CNN
+	1    11100 5100
 	1    0    0    1
 $EndComp
@@
 oscout
 $Comp
-L CONN_8 P7
+L CONN_8X2 P7
 U 1 1 5266B052
-P 5900 700
-F 0 "P7" V 5850 700 60  0000 C CNN
-F 1 "IN_1" V 5950 700 60  0000 C CNN
-F 2 "" H 5900 700 60  0000 C CNN
-F 3 "" H 5900 700 60  0000 C CNN
-	1    5900 700
-	0    -1   -1   0
-$EndComp
-$Comp
-L CONN_8 P8
+P 5900 650
+F 0 "P7" V 5850 650 60  0000 C CNN
+F 1 "IN_1" V 5950 650 60  0000 C CNN
+F 2 "" H 5900 650 60  0000 C CNN
+F 3 "" H 5900 650 60  0000 C CNN
+	1    5900 650
+	0    -1   -1   0
+$EndComp
+$Comp
+L CONN_8X2 P8
 U 1 1 5266B064
-P 6800 700
-F 0 "P8" V 6750 700 60  0000 C CNN
-F 1 "IN_2" V 6850 700 60  0000 C CNN
-F 2 "" H 6800 700 60  0000 C CNN
-F 3 "" H 6800 700 60  0000 C CNN
-	1    6800 700
-	0    -1   -1   0
-$EndComp
-$Comp
-L CONN_8 P9
+P 6800 650
+F 0 "P8" V 6750 650 60  0000 C CNN
+F 1 "IN_2" V 6850 650 60  0000 C CNN
+F 2 "" H 6800 650 60  0000 C CNN
+F 3 "" H 6800 650 60  0000 C CNN
+	1    6800 650
+	0    -1   -1   0
+$EndComp
+$Comp
+L CONN_8X2 P9
 U 1 1 5266B06F
-P 7700 700
-F 0 "P9" V 7650 700 60  0000 C CNN
-F 1 "IN_3" V 7750 700 60  0000 C CNN
-F 2 "" H 7700 700 60  0000 C CNN
-F 3 "" H 7700 700 60  0000 C CNN
-	1    7700 700
+P 7700 650
+F 0 "P9" V 7650 650 60  0000 C CNN
+F 1 "IN_3" V 7750 650 60  0000 C CNN
+F 2 "" H 7700 650 60  0000 C CNN
+F 3 "" H 7700 650 60  0000 C CNN
+	1    7700 650
 	0    -1   -1   0
 $EndComp
@@
 P 5650 6900
 F 0 "R4" V 5730 6900 50  0000 C CNN
-F 1 "R" V 5650 6900 50  0000 C CNN
+F 1 "770" V 5650 6900 50  0000 C CNN
 F 2 "" H 5650 6900 60  0000 C CNN
 F 3 "" H 5650 6900 60  0000 C CNN
@@
 P 5950 6900
 F 0 "R5" V 6030 6900 50  0000 C CNN
-F 1 "R" V 5950 6900 50  0000 C CNN
+F 1 "770" V 5950 6900 50  0000 C CNN
 F 2 "" H 5950 6900 60  0000 C CNN
 F 3 "" H 5950 6900 60  0000 C CNN
@@
 P 6250 6900
 F 0 "R6" V 6330 6900 50  0000 C CNN
-F 1 "R" V 6250 6900 50  0000 C CNN
+F 1 "770" V 6250 6900 50  0000 C CNN
 F 2 "" H 6250 6900 60  0000 C CNN
 F 3 "" H 6250 6900 60  0000 C CNN
@@
 P 6550 6900
 F 0 "R7" V 6630 6900 50  0000 C CNN
-F 1 "R" V 6550 6900 50  0000 C CNN
+F 1 "770" V 6550 6900 50  0000 C CNN
 F 2 "" H 6550 6900 60  0000 C CNN
 F 3 "" H 6550 6900 60  0000 C CNN
@@
 	2700 6500 2800 6600
 $Comp
-L CONN_4X2 P10
+L CONN_5X2 P10
 U 1 1 5266C027
 P 7800 5800
@@
 	1    0    0    -1
 $EndComp
-Text GLabel 8200 5950 2    60   Input ~ 0
-vss
-Text GLabel 7400 5650 0    60   Input ~ 0
+Text GLabel 8200 6000 2    60   Input ~ 0
+vss
+Text GLabel 7400 5700 0    60   Input ~ 0
 btn0
-Text GLabel 7400 5750 0    60   Input ~ 0
+Text GLabel 7400 5800 0    60   Input ~ 0
 btn1
-Text GLabel 7400 5850 0    60   Input ~ 0
+Text GLabel 7400 5900 0    60   Input ~ 0
 btn2
-Text GLabel 7400 5950 0    60   Input ~ 0
+Text GLabel 7400 6000 0    60   Input ~ 0
 btn3
 $Comp
@@
 P 9000 800
 F 0 "C8" H 9025 850 30  0000 L CNN
-F 1 "CSMALL" H 9025 750 30  0000 L CNN
+F 1 "100nF" H 9025 750 30  0000 L CNN
 F 2 "" H 9000 800 60  0000 C CNN
 F 3 "" H 9000 800 60  0000 C CNN
@@
 P 9000 1000
 F 0 "C9" H 9025 1050 30  0000 L CNN
-F 1 "CSMALL" H 9025 950 30  0000 L CNN
+F 1 "100nF" H 9025 950 30  0000 L CNN
 F 2 "" H 9000 1000 60  0000 C CNN
 F 3 "" H 9000 1000 60  0000 C CNN
@@
 P 9000 1200
 F 0 "C10" H 9025 1250 30  0000 L CNN
-F 1 "CSMALL" H 9025 1150 30  0000 L CNN
+F 1 "100nF" H 9025 1150 30  0000 L CNN
 F 2 "" H 9000 1200 60  0000 C CNN
 F 3 "" H 9000 1200 60  0000 C CNN
@@
 P 9000 1400
 F 0 "C11" H 9025 1450 30  0000 L CNN
-F 1 "CSMALL" H 9025 1350 30  0000 L CNN
+F 1 "100nF" H 9025 1350 30  0000 L CNN
 F 2 "" H 9000 1400 60  0000 C CNN
 F 3 "" H 9000 1400 60  0000 C CNN
@@
 P 9000 1600
 F 0 "C12" H 9025 1650 30  0000 L CNN
-F 1 "CSMALL" H 9025 1550 30  0000 L CNN
+F 1 "100nF" H 9025 1550 30  0000 L CNN
 F 2 "" H 9000 1600 60  0000 C CNN
 F 3 "" H 9000 1600 60  0000 C CNN
@@
 P 9400 800
 F 0 "C13" H 9425 850 30  0000 L CNN
-F 1 "CSMALL" H 9425 750 30  0000 L CNN
+F 1 "4.7uF" H 9425 750 30  0000 L CNN
 F 2 "" H 9400 800 60  0000 C CNN
 F 3 "" H 9400 800 60  0000 C CNN
@@
 P 9400 1000
 F 0 "C14" H 9425 1050 30  0000 L CNN
-F 1 "CSMALL" H 9425 950 30  0000 L CNN
+F 1 "100nF" H 9425 950 30  0000 L CNN
 F 2 "" H 9400 1000 60  0000 C CNN
 F 3 "" H 9400 1000 60  0000 C CNN
@@
 P 9400 1200
 F 0 "C15" H 9425 1250 30  0000 L CNN
-F 1 "CSMALL" H 9425 1150 30  0000 L CNN
+F 1 "1uF" H 9425 1150 30  0000 L CNN
 F 2 "" H 9400 1200 60  0000 C CNN
 F 3 "" H 9400 1200 60  0000 C CNN
@@
 P 9400 1400
 F 0 "C16" H 9425 1450 30  0000 L CNN
-F 1 "CSMALL" H 9425 1350 30  0000 L CNN
+F 1 "100nF" H 9425 1350 30  0000 L CNN
 F 2 "" H 9400 1400 60  0000 C CNN
 F 3 "" H 9400 1400 60  0000 C CNN
@@
 	0    -1   -1   0
 $EndComp
+Text GLabel 8900 800  0    60   Input ~ 0
+3v3
+Text GLabel 9500 800  2    60   Input ~ 0
+vss
+Text GLabel 7400 5600 0    60   Input ~ 0
+nrst
+Text GLabel 11500 2250 2    60   Input ~ 0
+12v
+NoConn ~ 4350 1650
+NoConn ~ 4250 1650
+NoConn ~ 3250 2950
+NoConn ~ 3250 4350
+NoConn ~ 3250 4450
 Wire Wire Line
 	8650 2150 8450 2150
@@
 Wire Wire Line
 	7350 2250 7700 2250
-Wire Wire Line
-	1150 4100 1900 4100
 Connection ~ 1400 4100
-Wire Wire Line
-	1150 4700 1900 4700
 Wire Wire Line
 	1400 4700 1400 4500
 Connection ~ 1400 4700
 Connection ~ 1750 4100
-Wire Wire Line
-	1150 4300 1150 4700
 Connection ~ 1750 4700
 Wire Bus Line
@@
 Wire Bus Line
 	2600 4850 3700 4850
-Wire Wire Line
-	8200 5650 8200 5950
-Connection ~ 8200 5750
-Connection ~ 8200 5850
 Wire Wire Line
 	9100 800  9100 1600
@@
 Connection ~ 8900 1200
 Connection ~ 8900 1000
-Text GLabel 8900 800  0    60   Input ~ 0
-3v3
-Text GLabel 9500 800  2    60   Input ~ 0
-vss
+Wire Wire Line
+	8200 5600 8200 6000
+Connection ~ 8200 5700
+Connection ~ 8200 5800
+Connection ~ 8200 5900
+Wire Wire Line
+	1400 4100 1900 4100
+Wire Wire Line
+	1400 4700 1900 4700
+Wire Wire Line
+	11500 2250 11500 5450
+Connection ~ 11500 5350
+Connection ~ 11500 5250
+Connection ~ 11500 5150
+Connection ~ 11500 5050
+Connection ~ 11500 4950
+Connection ~ 11500 4850
+Connection ~ 11500 4750
+Connection ~ 11500 4200
+Connection ~ 11500 4100
+Connection ~ 11500 4000
+Connection ~ 11500 3900
+Connection ~ 11500 3800
+Connection ~ 11500 3700
+Connection ~ 11500 3600
+Connection ~ 11500 2850
+Connection ~ 11500 2750
+Connection ~ 11500 2650
+Connection ~ 11500 2550
+Connection ~ 11500 2450
+Connection ~ 11500 2350
+Connection ~ 11500 3500
+Connection ~ 11500 2950
+Text GLabel 5550 250  0    60   Input ~ 0
+vss
+Wire Wire Line
+	5550 250  8050 250
+Connection ~ 5650 250
+Connection ~ 5750 250
+Connection ~ 5850 250
+Connection ~ 5950 250
+Connection ~ 6050 250
+Connection ~ 6150 250
+Connection ~ 6250 250
+Connection ~ 6450 250
+Connection ~ 6550 250
+Connection ~ 6650 250
+Connection ~ 6750 250
+Connection ~ 6850 250
+Connection ~ 6950 250
+Connection ~ 7050 250
+Connection ~ 7150 250
+Connection ~ 7350 250
+Connection ~ 7450 250
+Connection ~ 7550 250
+Connection ~ 7650 250
+Connection ~ 7750 250
+Connection ~ 7850 250
+Connection ~ 7950 250
 $EndSCHEMATC

Commit message: WIP: host PCB
Parts:
- removed P12: PWR_OUT, symbol CONN_2
- R3: value R -> 770
Connections:
- wire segments 78 -> 80
Other:
- moved on the sheet: U2, U3, U4
